File: keyboard-pcb/keyboard-pcb.kicad_pcb (KiCad board)
At the start: 2 copper layers, 304.8 x 114.3 mm, 379 parts, among them Q1 Q_Photo_NPN, Q10 Q_Photo_NPN, Q11 Q_Photo_NPN, Q12 Q_Photo_NPN, Q13 Q_Photo_NPN, Q14 Q_Photo_NPN, Q15 Q_Photo_NPN, Q16 Q_Photo_NPN, Q17 Q_Photo_NPN, Q18 Q_Photo_NPN, Q19 Q_Photo_NPN, Q2 Q_Photo_NPN, Q20 Q_Photo_NPN, Q21 Q_Photo_NPN, Q22 Q_Photo_NPN, Q23 Q_Photo_NPN, Q24 Q_Photo_NPN, Q25 Q_Photo_NPN, Q26 Q_Photo_NPN, Q27 Q_Photo_NPN, Q28 Q_Photo_NPN, Q29 Q_Photo_NPN, Q3 Q_Photo_NPN, Q30 Q_Photo_NPN, Q31 Q_Photo_NPN, Q32 Q_Photo_NPN, Q33 Q_Photo_NPN, Q34 Q_Photo_NPN, Q35 Q_Photo_NPN, Q36 Q_Photo_NPN, Q37 Q_Photo_NPN, Q38 Q_Photo_NPN, Q39 Q_Photo_NPN, Q4 Q_Photo_NPN, Q40 Q_Photo_NPN, Q41 Q_Photo_NPN, Q42 Q_Photo_NPN, Q43 Q_Photo_NPN, Q44 Q_Photo_NPN, Q45 Q_Photo_NPN, Q46 Q_Photo_NPN, Q47 Q_Photo_NPN, Q48 Q_Photo_NPN, Q49 Q_Photo_NPN, Q5 Q_Photo_NPN, Q50 Q_Photo_NPN, Q51 Q_Photo_NPN, Q52 Q_Photo_NPN, Q53 Q_Photo_NPN, Q54 Q_Photo_NPN, Q55 Q_Photo_NPN, Q56 Q_Photo_NPN, Q57 Q_Photo_NPN, Q58 Q_Photo_NPN, Q59 Q_Photo_NPN, Q6 Q_Photo_NPN, Q60 Q_Photo_NPN, Q61 Q_Photo_NPN, Q62 Q_Photo_NPN, Q63 Q_Photo_NPN, Q64 Q_Photo_NPN, Q65 Q_Photo_NPN, Q66 Q_Photo_NPN, Q67 Q_Photo_NPN, Q68 Q_Photo_NPN, Q69 Q_Photo_NPN, Q7 Q_Photo_NPN, Q70 Q_Photo_NPN, Q71 Q_Photo_NPN, Q72 Q_Photo_NPN, Q73 Q_Photo_NPN, Q74 Q_Photo_NPN, Q75 Q_Photo_NPN, Q8 Q_Photo_NPN, Q9 Q_Photo_NPN, U1 BlackPill

Commit message: Fixed outlines of edgecuts
 M .gitignore
A  Optical_Parts.pretty/MountingHole_2.2mm_M2.kicad_mod
M  keyboard-pcb/keyboard-pcb.kicad_pcb
M  keyboard-pcb/keyboard-pcb.kicad_prl
M  switch-cutout/switch-cutout.kicad_pcb
M  switch-cutout/switch-cutout.kicad_prl
Parts:
- removed the REF** at (280.4, 39.8)
- added REF**: MountingHole_1.2mm_M1, OpticalParts:MountingHole_1.2mm_M1, F.Cu at (204.8, 47.6)
- added REF**: MountingHole_2.2mm_M2, OpticalParts:MountingHole_2.2mm_M2, F.Cu at (128.6, 47.6)
- added REF**: MountingHole_1.2mm_M1, OpticalParts:MountingHole_1.2mm_M1, F.Cu at (266.7, 28.6)
- added REF**: MountingHole_1.2mm_M1, OpticalParts:MountingHole_1.2mm_M1, F.Cu at (7.14, 47.6)
- added REF**: MountingHole_2.2mm_M2, OpticalParts:MountingHole_2.2mm_M2, F.Cu at (152.4, 9.53)
- added REF**: MountingHole_2.2mm_M2, OpticalParts:MountingHole_2.2mm_M2, F.Cu at (90.5, 47.6)
- added REF**: MountingHole_2.2mm_M2, OpticalParts:MountingHole_2.2mm_M2, F.Cu at (52.4, 66.7)
- added REF**: MountingHole_2.2mm_M2, OpticalParts:MountingHole_2.2mm_M2, F.Cu at (76.2, 28.6)
- added REF**: MountingHole_2.2mm_M2, OpticalParts:MountingHole_2.2mm_M2, F.Cu at (57.1, 9.53)
- added REF**: MountingHole_2.2mm_M2, OpticalParts:MountingHole_2.2mm_M2, F.Cu at (7.14, 57.1)
- added REF**: MountingHole_2.2mm_M2, OpticalParts:MountingHole_2.2mm_M2, F.Cu at (190.5, 28.6)
- added REF**: MountingHole_2.2mm_M2, OpticalParts:MountingHole_2.2mm_M2, F.Cu at (269.1, 11.9)
- added REF**: MountingHole_2.2mm_M2, OpticalParts:MountingHole_2.2mm_M2, F.Cu at (266.7, 64.3)
- added REF**: MountingHole_2.2mm_M2, OpticalParts:MountingHole_2.2mm_M2, F.Cu at (21.4, 38.1)
- added REF**: MountingHole_2.2mm_M2, OpticalParts:MountingHole_2.2mm_M2, F.Cu at (169.1, 69.1)
- added REF**: MountingHole_2.2mm_M2, OpticalParts:MountingHole_2.2mm_M2, F.Cu at (228.6, 66.7)
- added REF**: MountingHole_1.2mm_M1, OpticalParts:MountingHole_1.2mm_M1, F.Cu at (71.4, 66.7)
- added REF**: MountingHole_2.2mm_M2, OpticalParts:MountingHole_2.2mm_M2, F.Cu at (228.6, 28.6)
- added REF**: MountingHole_2.2mm_M2, OpticalParts:MountingHole_2.2mm_M2, F.Cu at (107.2, 69.1)
- added REF**: MountingHole_2.2mm_M2, OpticalParts:MountingHole_2.2mm_M2, F.Cu at (281.0, 38.1)
Routing:
- net /col15: track 467.0 -> 497.4 mm, vias 11 -> 15
- net /col14: track 314.2 -> 317.8 mm
- net /col13: track 342.8 -> 345.9 mm
- net /row5: track 376.1 -> 378.8 mm
- net /col12: track 364.4 -> 366.9 mm
- net /col4: track 200.4 -> 202.8 mm
- net /col11: track 308.9 -> 310.9 mm
- net /col10: track 292.3 -> 293.8 mm
- net /row2: track 381.6 -> 382.8 mm
Other:
- outline, holes or cut-outs redrawn
