File: switch-cutout/switch-cutout.kicad_pcb (KiCad board)
At the start: 2 copper layers, 16.9 x 16.9 mm, 80 parts

Commit message: Fixed outlines of edgecuts
 M .gitignore
A  Optical_Parts.pretty/MountingHole_2.2mm_M2.kicad_mod
M  keyboard-pcb/keyboard-pcb.kicad_pcb
M  keyboard-pcb/keyboard-pcb.kicad_prl
M  switch-cutout/switch-cutout.kicad_pcb
M  switch-cutout/switch-cutout.kicad_prl
Parts:
- added ?: , clipboard:7bfbbc5f-3758-4a9b-ae23-8507aae1abe4, F.Cu at (150.6, 114.2)
- added REF**: TestPoint_THTPad_1.0x1.0mm_Drill0.5mm, TestPoint:TestPoint_THTPad_1.0x1.0mm_Drill0.5mm, F.Cu at (142.1, 109.6)
- added REF**: MountingHole_2.2mm_M2, OpticalParts:MountingHole_2.2mm_M2, F.Cu at (276.2, 81.0)
- added REF**: MountingHole_2.2mm_M2, OpticalParts:MountingHole_2.2mm_M2, F.Cu at (16.7, 81.0)
- added REF**: TestPoint_THTPad_1.0x1.0mm_Drill0.5mm, TestPoint:TestPoint_THTPad_1.0x1.0mm_Drill0.5mm, F.Cu at (155.1, 109.7)
- added REF**: R_Axial_DIN0204_L3.6mm_D1.6mm_P7.62mm_Horizontal, Resistor_THT:R_Axial_DIN0204_L3.6mm_D1.6mm_P7.62mm_Horizontal, F.Cu at (145.0, 116.0)
- added REF**: MountingHole_2.2mm_M2, OpticalParts:MountingHole_2.2mm_M2, F.Cu at (123.8, 90.5)
- added REF**: MountingHole_2.2mm_M2, OpticalParts:MountingHole_2.2mm_M2, F.Cu at (52.4, 52.4)
- added REF**: MountingHole_2.2mm_M2, OpticalParts:MountingHole_2.2mm_M2, F.Cu at (223.8, 71.4)
- added REF**: MountingHole_2.2mm_M2, OpticalParts:MountingHole_2.2mm_M2, F.Cu at (71.4, 71.4)
- added REF**: MountingHole_2.2mm_M2, OpticalParts:MountingHole_2.2mm_M2, F.Cu at (261.9, 107.2)
- added REF**: MountingHole_2.2mm_M2, OpticalParts:MountingHole_2.2mm_M2, F.Cu at (264.3, 54.8)
- added REF**: MountingHole_2.2mm_M2, OpticalParts:MountingHole_2.2mm_M2, F.Cu at (2.38, 100.0)
- added REF**: MountingHole_1.2mm_M1, OpticalParts:MountingHole_1.2mm_M1, F.Cu at (28.6, 109.5)
- added REF**: MountingHole_1.2mm_M1, OpticalParts:MountingHole_1.2mm_M1, F.Cu at (128.6, 52.4)
- added REF**: MountingHole_2.2mm_M2, OpticalParts:MountingHole_2.2mm_M2, F.Cu at (47.6, 109.5)
- added REF**: MountingHole_2.2mm_M2, OpticalParts:MountingHole_2.2mm_M2, F.Cu at (147.6, 52.4)
- added REF**: MountingHole_2.2mm_M2, OpticalParts:MountingHole_2.2mm_M2, F.Cu at (85.7, 90.5)
- added REF**: MountingHole_2.2mm_M2, OpticalParts:MountingHole_2.2mm_M2, F.Cu at (102.4, 111.9)
- added REF**: MountingHole_2.2mm_M2, OpticalParts:MountingHole_2.2mm_M2, F.Cu at (185.7, 71.4)
- added REF**: MountingHole_2.2mm_M2, OpticalParts:MountingHole_2.2mm_M2, F.Cu at (223.8, 109.5)
- added REF**: MountingHole_2.2mm_M2, OpticalParts:MountingHole_2.2mm_M2, F.Cu at (164.3, 111.9)
- added REF**: MountingHole_1.2mm_M1, OpticalParts:MountingHole_1.2mm_M1, F.Cu at (33.3, 52.4)
- added REF**: MountingHole_1.2mm_M1, OpticalParts:MountingHole_1.2mm_M1, F.Cu at (252.4, 52.4)
- added REF**: MountingHole_1.2mm_M1, OpticalParts:MountingHole_1.2mm_M1, F.Cu at (242.9, 109.5)
- moved ? 61.5 mm to (119.2, 113.8)
- moved REF** 61.5 mm to (113.6, 115.5)
- moved REF** 61.5 mm to (110.7, 109.1)
- moved REF** 61.5 mm to (123.7, 109.2)
Routing:
- net (no net): track 21.4 -> 41.4 mm
Other:
- board size 16.9 x 16.9 mm -> 304.8 x 114.3 mm
